Commit message: Added ground plane to urdf

File: urdf/ur.urdf.xacro (robot description, xacro)
@@ -51,4 +51,26 @@
    <!-- create link fixed to the "world" -->
    <link name="world" />
+   <link name="ground_plane">
+     <visual>
+       <origin rpy="0 0 0" xyz="0 0 0"/>
+       <geometry>
+         <box size="5 5 0"/>
+       </geometry>
+       <material name="ground_white">
+         <color rgba="1 1 1 0.5"/>
+       </material>
+     </visual>
+     <collision>
+       <origin rpy="0 0 0" xyz="0 0 0"/>
+       <geometry>
+         <box size="5 5 0"/>
+       </geometry>
+     </collision>
+   </link>
+   <joint name="ground_plane_joint" type="fixed">
+     <origin xyz="0 0 -0.01" rpy="0 0 0"/>
+     <parent link="world"/>
+     <child link="ground_plane"/>
+   </joint>
    <!-- arm -->
    <xacro:ur_robot

Commit message: Added condition on simulation for ground plane

File: urdf/ur.urdf.xacro (robot description, xacro)
@@ -49,28 +49,32 @@
    <!-- convert to property to use substitution in function -->
    <xacro:property name="initial_positions_file" default="$(arg initial_positions_file)"/>
+   <xacro:property name="is_sim_gazebo" value="$(arg sim_gazebo)"/>
+   <xacro:property name="is_sim_ignition" value="$(arg sim_ignition)"/>
    <!-- create link fixed to the "world" -->
    <link name="world" />
-   <link name="ground_plane">
-     <visual>
-       <origin rpy="0 0 0" xyz="0 0 0"/>
-       <geometry>
-         <box size="5 5 0"/>
-       </geometry>
-       <material name="ground_white">
-         <color rgba="1 1 1 0.5"/>
-       </material>
-     </visual>
-     <collision>
-       <origin rpy="0 0 0" xyz="0 0 0"/>
-       <geometry>
-         <box size="5 5 0"/>
-       </geometry>
-     </collision>
-   </link>
-   <joint name="ground_plane_joint" type="fixed">
-     <origin xyz="0 0 -0.01" rpy="0 0 0"/>
-     <parent link="world"/>
-     <child link="ground_plane"/>
-   </joint>
+   <xacro:if value="${is_sim_gazebo or is_sim_ignition}">
+     <link name="ground_plane">
+       <visual>
+         <origin rpy="0 0 0" xyz="0 0 0"/>
+         <geometry>
+           <box size="5 5 0"/>
+         </geometry>
+         <material name="ground_white">
+           <color rgba="1 1 1 0.5"/>
+         </material>
+       </visual>
+       <collision>
+         <origin rpy="0 0 0" xyz="0 0 0"/>
+         <geometry>
+           <box size="5 5 0"/>
+         </geometry>
+       </collision>
+     </link>
+     <joint name="ground_plane_joint" type="fixed">
+       <origin xyz="0 0 -0.01" rpy="0 0 0"/>
+       <parent link="world"/>
+       <child link="ground_plane"/>
+     </joint>
+   </xacro:if>
    <!-- arm -->
    <xacro:ur_robot
